Commit message: RTABMapping launch file and changes to robot urdf

File: src/my_robot/urdf/my_robot.xacro (robot description, xacro)
@@ -111,4 +111,6 @@
     </visual>
   </link>
+  <link name="optical_camera">
+  </link>
   <link name="hokuyo">
     <pose>0 0 0 0 0 0</pose>
@@ -165,4 +167,9 @@
     <axis xyz="0 1 0" rpy="0 0 0" />
   </joint>
+  <joint name="optical_camera_joint" type="fixed">
+    <origin xyz="0 0 0" rpy="-1.5707 0 -1.5707" />
+    <parent link="camera" />
+    <child link="optical_camera" />
+  </joint>
 <!-- GAZEBO ELEMENTS -->
   <gazebo reference="left_wheel">
